File: EnvChocTKL.kicad_pcb (KiCad board)
At the start: 2 copper layers, 340 x 112 mm, 181 parts, among them U1 EliteC

Commit message: added mount holes, a few silkscreen marks and generated revision 0 gerber
Parts:
- added H1: MountingHole_Pad, MountingHole:MountingHole_2.5mm_Pad, F.Cu at (55.2, 134.2)
- added H2: MountingHole_Pad, MountingHole:MountingHole_2.5mm_Pad, F.Cu at (55.4, 217.7)
- added H3: MountingHole_Pad, MountingHole:MountingHole_2.5mm_Pad, F.Cu at (317.5, 153.3)
- added H4: MountingHole_Pad, MountingHole:MountingHole_2.5mm_Pad, F.Cu at (370.3, 216.0)
- moved U1 0.90 mm to (192.2, 226.0)
Routing:
- net col6: track 171.4 -> 151.4 mm
- net row0: track 420.7 -> 417.5 mm
- net col14: track 241.0 -> 244.0 mm
- net col13: track 216.8 -> 219.7 mm
- net col12: track 197.0 -> 200.0 mm
- net col4: track 210.5 -> 208.0 mm
- net col5: track 174.8 -> 172.4 mm
- net col15: track 259.6 -> 262.1 mm
- net col11: track 199.1 -> 201.4 mm
- net row2: track 376.1 -> 377.6 mm
- net row5: track 326.9 -> 325.5 mm
- net col10: track 170.2 -> 171.5 mm
- net col1: track 254.3 -> 253.3 mm
- net row1: track 401.7 -> 400.7 mm
- net col0: track 293.9 -> 293.0 mm
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Other:
- board text added: "https://github.com/Envious-Data/Env-ChocV2TKL Rev#0 Concept board."
- board text added: "the microcontroller goes on the other side of this PCB You need an Elite-C/Puchi-C"
