File: EnvChocTKL.kicad_pcb (KiCad board)
At the start: 2 copper layers, 340 x 112 mm, 185 parts, among them U1 EliteC

Commit message: Corrected some errors and generated a fixed gerber
Routing:
- net row0: track 417.5 -> 418.3 mm
- net col5: track 172.4 -> 171.7 mm

Commit message: swapped footprint to sort of fit chocV1 as well and corrected all DRC errors
Routing:
- net col3: track 237.5 -> 245.4 mm
- net col4: track 208.1 -> 215.3 mm
- net col6: track 151.2 -> 156.7 mm
- net col5: track 171.7 -> 176.4 mm
- net col10: track 171.5 -> 176.1 mm
- net col8: track 154.2 -> 158.8 mm
- net col2: track 237.5 -> 240.4 mm
- net col13: track 219.7 -> 222.6 mm
- net col1: track 253.5 -> 256.1 mm
- net col9: track 172.2 -> 174.8 mm
- net col11: track 201.4 -> 203.3 mm
- net Net-(D_32-Pad2): track 18.3 -> 19.9 mm
- net col0: track 293.0 -> 294.6 mm
- net row0: track 418.3 -> 419.8 mm
- net col14: track 244.0 -> 245.5 mm
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
Commit message: replaced stabs with cutouts for lower profile mounting and fixed issues relating to such, generated updated gerber
Parts:
- removed Stab1, Stab2, Stab3: MountingHole_Pad, Mounting_Keyboard_Stabilizer:Stabilizer_Cherry_MX_2u
- removed Stab4: MountingHole_Pad, Mounting_Keyboard_Stabilizer:Stabilizer_Cherry_MX_6.25u
- moved H3 6.69 mm to (318.2, 146.6)
- moved D_75 5.62 mm to (297.5, 216.0)
Routing:
- net col4: track 215.3 -> 182.7 mm
- net col14: track 245.5 -> 269.9 mm
- net col3: track 245.4 -> 225.0 mm
- net col12: track 199.8 -> 208.7 mm
- net col11: track 203.3 -> 212.2 mm
- net col10: track 176.1 -> 184.9 mm
- net row4: track 363.9 -> 370.4 mm
- net Net-(D_75-Pad2): track 4.48 -> 10.3 mm
- net col13: track 222.6 -> 227.0 mm
- net row3: track 315.5 -> 319.3 mm
- net col15: track 262.1 -> 265.7 mm
- net col2: track 240.4 -> 244.0 mm
- net col0: track 294.6 -> 298.2 mm
- net col1: track 256.1 -> 259.7 mm
- net row2: track 379.1 -> 376.5 mm
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Other:
- outline, holes or cut-outs redrawn

Commit message: changed cutout shape and generated another gerber
Routing:
- net row1: track 400.6 -> 399.1 mm
- net Net-(D_75-Pad2): track 10.3 -> 9.06 mm
- net row2: track 376.5 -> 375.5 mm
- net col2: track 244.0 -> 243.4 mm
Other:
- outline, holes or cut-outs redrawn

Commit message: moved MCU and redid a bunch of traces
Parts:
- removed H1, H2, H3: MountingHole_Pad, MountingHole:MountingHole_2.5mm_Pad
- K_0, K_1, K_10, K_11, K_12, K_13, K_14, K_15, K_16, K_17, K_18, K_19, K_2, K_20, K_21, K_22, K_23, K_24, K_25, K_26, K_27, K_28, K_3, K_30, K_31, K_32, K_34, K_35, K_36, K_37, K_38, K_39, K_4, K_40, K_41, K_42, K_43, K_44, K_45, K_47, K_48, K_49, K_5, K_51, K_52, K_53, K_54, K_55, K_56, K_57, K_58, K_59, K_6, K_60, K_61, K_62, K_64, K_65, K_66, K_67, K_68, K_69, K_7, K_70, K_71, K_72, K_73, K_74, K_76, K_8, K_85, K_86, K_87, K_9: footprint Switch_Keyboard_Kailh:SW_Kailh_Choc_V2 -> Switch_Keyboard_Kailh:SW_Kailh_Choc_V1_1.00u
- K_29: footprint Switch_Keyboard_Kailh:SW_Kailh_Choc_V2 -> Switch_Keyboard_Kailh:SW_Kailh_Choc_V1_2.00u
- K_33: footprint Switch_Keyboard_Kailh:SW_Kailh_Choc_V2 -> Switch_Keyboard_Kailh:SW_Kailh_Choc_V1_1.50u
- K_46: footprint Switch_Keyboard_Kailh:SW_Kailh_Choc_V2 -> Switch_Keyboard_Kailh:SW_Kailh_Choc_V1_ISOEnter
- K_50: footprint Switch_Keyboard_Kailh:SW_Kailh_Choc_V2 -> Switch_Keyboard_Kailh:SW_Kailh_Choc_V1_1.75u
- K_63, K_77, K_78, K_79, K_81, K_82, K_83, K_84: footprint Switch_Keyboard_Kailh:SW_Kailh_Choc_V2 -> Switch_Keyboard_Kailh:SW_Kailh_Choc_V1_1.25u
- K_75: footprint Switch_Keyboard_Kailh:SW_Kailh_Choc_V2 -> Switch_Keyboard_Kailh:SW_Kailh_Choc_V1_2.75u
- K_80: footprint Switch_Keyboard_Kailh:SW_Kailh_Choc_V2 -> Switch_Keyboard_Kailh:SW_Kailh_Choc_V1_6.25u
- moved U1 186.5 mm to (354.1, 133.4)
- moved D_14 46.7 mm to (309.1, 136.9)
- moved D_12 46.6 mm to (271.1, 137.0)
- moved D_13 46.6 mm to (290.1, 136.9)
- moved D_9 46.6 mm to (213.9, 137.0)
- moved D_11 46.6 mm to (252.0, 137.0)
- moved D_10 46.6 mm to (233.0, 137.1)
- moved D_15 44.1 mm to (314.2, 136.2)
- moved K_11 41.3 mm to (248.9, 134.3)
- moved K_10 41.2 mm to (229.8, 134.3)
- moved K_12 41.2 mm to (267.9, 134.3)
- moved K_13 41.2 mm to (287.0, 134.3)
- moved K_14 41.2 mm to (306.0, 134.3)
- moved K_15 41.2 mm to (325.1, 134.3)
- moved K_9 41.2 mm to (210.8, 134.3)
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Connections:
- U1 pad 1: col0 -> col17
- U1 pad 10: col7 -> col10
- U1 pad 11: col8 -> col9
- U1 pad 12: col9 -> col8
- U1 pad 13: col15 -> col2
- U1 pad 14: col16 -> col1
- U1 pad 15: col17 -> col0
- U1 pad 2: col1 -> col16
- U1 pad 21: Net-(U1-Pad21) -> (no net)
- U1 pad 22: Net-(U1-Pad22) -> (no net)
- U1 pad 25: col10 -> col7
- U1 pad 26: col11 -> col6
- U1 pad 27: col12 -> col5
- U1 pad 28: col13 -> col4
- U1 pad 29: col14 -> col3
- U1 pad 5: col2 -> col15
- U1 pad 6: col3 -> col14
- U1 pad 7: col4 -> col13
- U1 pad 8: col5 -> col12
- U1 pad 9: col6 -> col11
Routing:
- net col3: track 225.0 -> 383.3 mm
- net col4: track 182.7 -> 337.4 mm
- net col1: track 259.4 -> 411.2 mm
- net col7: track 146.9 -> 294.3 mm
- net col2: track 243.4 -> 382.8 mm
- net col5: track 176.4 -> 313.0 mm, vias 1 -> 0
- net col6: track 156.7 -> 282.1 mm, vias 1 -> 0
- net col0: track 297.9 -> 415.6 mm
- net col8: track 158.8 -> 271.8 mm
- net row5: track 325.1 -> 431.3 mm, vias 3 -> 0
- net row0: track 418.0 -> 319.2 mm, vias 1 -> 0
- net col15: track 265.7 -> 173.6 mm
- net col9: track 174.8 -> 254.7 mm
- net row3: track 319.3 -> 397.0 mm, vias 1 -> 0
- net col10: track 185.2 -> 256.5 mm
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Other:
- board size 340 x 112 mm -> 343.3 x 115.1 mm

Commit message: added mount holes and adjusted some traces in relation
Parts:
- added H1: MountingHole_Pad, MountingHole:MountingHole_2.5mm_Pad, F.Cu at (318.4, 162.7)
- added H2: MountingHole_Pad, MountingHole:MountingHole_2.5mm_Pad, F.Cu at (51.7, 143.9)
- added H3: MountingHole_Pad, MountingHole:MountingHole_2.5mm_Pad, F.Cu at (56.6, 220.2)
Routing:
- net row3: track 397.0 -> 394.2 mm
- net col1: track 411.2 -> 413.8 mm
- net col17: track 231.4 -> 229.2 mm
- net col15: track 173.6 -> 171.8 mm
- net row1: track 375.9 -> 376.8 mm
- net row5: track 431.3 -> 430.7 mm
- net GND: vias 5 -> 3

Commit message: updated silkscreen and ran cleanup
Routing:
- net Net-(D_12-Pad2): track 6.34 -> 0.00 mm
- net row1: track 376.8 -> 378.1 mm
Other:
- board text added: "https://github.com/Envious-Data/Env-ChocV2TKL Revision 16"
- board text removed: "https://github.com/Envious-Data/Env-ChocV2TKL Rev#0 Concept board."
