File: EnvChocTKL.kicad_sch (KiCad schematic)
At the start: 227 parts, among them J2 SKRKAEE020, J5 Conn_01x03_Male, Q1 Si2329DS, U1 TLV75533PDBVR, U3 RP2040, Y1 3225_4P

Commit message: Swapped MCU from onboard RP2040 to RPI PICO
Parts:
- removed C1: 10uf 402, Capacitor_SMD:C_0402_1005Metric, symbol Device:C
- removed C10, C3: 1uf 0201, Capacitor_SMD:C_0201_0603Metric, symbol Device:C
- removed C11, C13, C14, C15, C16, C18, C5, C6, C7, C8: 100nf 0201, Capacitor_SMD:C_0201_0603Metric, symbol Device:C
- removed C17, C4, CBP1: 10uf 0402, Capacitor_SMD:C_0402_1005Metric, symbol Device:C
- removed C19, C2: 22pf 0402, Capacitor_SMD:C_0402_1005Metric, symbol Device:C
- removed F1: 0805L050WR, Fuse:Fuse_0805_2012Metric, symbol Device:Polyfuse_Small
- removed FLASH1: W25Q16JVSSIQ, Package_SO:SOIC-8_5.23x5.23mm_P1.27mm, symbol W25Q256JVEIQ_TR:W25Q256JVEIQ_TR
- removed GPIO24_LED1, GPIO25_LED1: LED_0402, LED_SMD:LED_0402_1005Metric, symbol Device:LED
- removed GPIO24_RESISTOR1, GPIO25_RESISTOR1: 470 0402 Resistor, Resistor_SMD:R_0402_1005Metric, symbol Device:R
- removed J2, RSW1: SKRKAEE020, Button_Switch_SMD:SW_Push_SPST_NO_Alps_SKRK, symbol Switch:SW_Push
- removed J5: Conn_01x03_Male, TestPoint:TestPoint_2Pads_Pitch2.54mm_Drill0.8mm, symbol Connector_Generic:Conn_01x03
- removed NT1: NetTie_2, NetTie:NetTie-2_SMD_Pad0.5mm, symbol Device:NetTie_2
- removed Q1: Si2329DS, Package_TO_SOT_SMD:SOT-23, symbol Transistor_FET:Si2319CDS
- removed R1, R11: 1K 0201, Resistor_SMD:R_0201_0603Metric, symbol Device:R
- removed R10: 1 0402, Resistor_SMD:R_0402_1005Metric, symbol Device:R_Small
- removed R2: 10K 0402, Resistor_SMD:R_0402_1005Metric, symbol Device:R
- removed R3, R4: 27 0402 Resistor, Resistor_SMD:R_0402_1005Metric, symbol Device:R
- removed R7: 100K 0402 resistor, Resistor_SMD:R_0402_1005Metric, symbol Device:R
- removed R9: 200 0603, Resistor_SMD:R_0603_1608Metric, symbol Device:R_Small
- removed U1: TLV75533PDBVR, Package_TO_SOT_SMD:SOT-23-5, symbol Regulator_Linear:AP131-15
- removed U3: RP2040, RP2040_minimal:RP2040-QFN-56, symbol MCU_RaspberryPi_RP2040:RP2040
- removed Y1: 3225_4P, Crystal:Crystal_SMD_3225-4Pin_3.2x2.5mm, symbol Device:Crystal_GND24
- added RPI1: Pico, MCU_RaspberryPi_and_Boards:RPi_Pico_SMD_TH_MODIFIED, symbol PicoModified:Pico
Connections:
- net GND: now also RPI1.13 (GND), RPI1.18 (GND), RPI1.23 (GND), RPI1.28 (GND), RPI1.3 (GND), RPI1.33 (AGND), RPI1.38 (GND), RPI1.8 (GND), RPI1.TP1 (GND_L)
- net USB_D+: now also RPI1.TP3 (USB_DP)
- net USB_D-: now also RPI1.TP2 (USB_DM)
- net col0: now also RPI1.21 (GPIO16)
- net col1: now also RPI1.22 (GPIO17)
- net col10: now also RPI1.17 (GPIO13)
- net col11: now also RPI1.16 (GPIO12)
- net col12: now also RPI1.15 (GPIO11)
- net col13: now also RPI1.14 (GPIO10)
- net col14: now also RPI1.12 (GPIO9)
- net col15: now also RPI1.11 (GPIO8)
- net col16: now also RPI1.10 (GPIO7)
- net col17: now also RPI1.9 (GPIO6)
- net col2: now also RPI1.24 (GPIO18)
- net col3: now also RPI1.25 (GPIO19)
- net col4: now also RPI1.26 (GPIO20)
- net col5: now also RPI1.27 (GPIO21)
- net col6: now also RPI1.29 (GPIO22)
- net col7: now also RPI1.31 (GPIO26_ADC0)
- net col8: now also RPI1.20 (GPIO15)
- net col9: now also RPI1.19 (GPIO14)
- net row0: now also RPI1.7 (GPIO5)
- net row1: now also RPI1.6 (GPIO4)
- net row2: now also RPI1.5 (GPIO3)
- net row3: now also RPI1.4 (GPIO2)
- net row4: now also RPI1.2 (GPIO1)
- net row5: now also RPI1.1 (GPIO0)
Other:
- note removed: "1K resistor to prevent overdriving of the crystal as per the minimal design example"
- note removed: "500mA hold current 1A trip 6V trip"
- note removed: "Crystal"
- note removed: "D1 NEEDS to be 0omh resistor or 1N4002 diode"
- note removed: "Flash"
- note removed: "GD25Q40CEIGR is NOT Compatible you need GD25W16* needs to be a multiple of 8 atleast for circuitpython. (Ive not confirmed if GD25W16 works I just Have some boards with GD25Q40CEIGR and they dont work)"
- note removed: "GPIOs"
- note removed: "Im pretty sure a lot of these W25QXXX Chips are pin compatible Dont quote me on that"
- note removed: "Im unsure if the RP2040 can function with flash larger than 128Mb"
- note removed: "KoreanHROParts USB_C_Receptacle_HRO_TYPE-C-31-M-12"
- note removed: "LEDs"
- note removed: "MAKE SURE THIS LINE is ran off of pin43 or close to pin43"
- note removed: "Make sure C10 is close to pin 44 of RP2040"
- note removed: "Make sure C3 is close to pin 45 of RP2040"
- note removed: "Make sure R3 and R4 are close to RP2040"
- note removed: "Make sure the flash chip you have selected supports 3.3V power or adjust the design."
- note removed: "Only fit cBP1 if you have selected an alternate voltage regulator TLV75533PDBVR does not require cBP1."
- note removed: "Pin 9 technically doesnt exist its the main central contact under the chip for heat dicipation"
- note removed: "Power LED is on by default but when GPIO24 is enabled it will be shut off"
- note removed: "RP2040 supports 1MHz to 15MHz"
- note removed: "These decoupling capacitors are meant to be put close by each 3.3V pin of the RP2040"
- note removed: "Would assume you could just not connect SD2 and SD3 for non QSPI"
- note removed: "https://datasheets.raspberrypi.com/rp2040/hardware-design-with-rp2040.pdf On page 13 you can learn more details of what flash is supported"
- note removed: "not 22pf but pick to match crystal."
- note removed: "suposedly the rp2040 supports SPI-2 flash but I havent tried it."
- note removed: "this is for factory testing always pull this to ground"
